File: SpringRobocon2026_mainboard.kicad_sch (KiCad schematic)
At the start: 63 parts, among them J1 Conn_01x05_Socket_Encoder1, J10 Conn_01x05_Socket_Encoder5, J2 Conn_01x05_Socket_Encoder3, J3 FDCAN_1, J4 Conn_01x05_Socket_Encoder2, J5 Conn_01x05_Socket_Encoder4, J6 FDCAN_2, J7 Conn_01x03_Pin, J8 Conn_01x04_Pin, J9 Conn_01x03_Pin, SW3 SW_DIP_x02_CANnum, U1 XT60_M, U2 MCP2562-E-P, U3 BP5293-50, U4 BA033CC0FP, U5 MCP2562-E-P, U6 NUCLEO-F446RE, U7 XT60_M

Commit message: 回路図完成した
Parts:
- removed J9: Conn_01x03_Pin, Connector_JST:JST_XH_B3B-XH-A_1x03_P2.50mm_Vertical, symbol Connector:Conn_01x03_Pin
- removed U7: XT60_M, Connector_AMASS:AMASS_XT60-M_1x02_P7.20mm_Vertical, symbol Mylib:XT60
- added J11: Conn_01x03_Pin, Connector_JST:JST_XH_B3B-XH-A_1x03_P2.50mm_Vertical, symbol Connector:Conn_01x03_Pin
- added J8: Conn_01x03_Pin, Connector_PinHeader_2.54mm:PinHeader_1x03_P2.54mm_Vertical, symbol Connector:Conn_01x03_Pin
- U2, U5: value MCP2562-E-P -> ATA6561; footprint Package_DIP:DIP-8_W7.62mm -> MyLib:ATA6561
- renumbered C9 to C10, C10 to C14, C14 to C15, C15 to C16, C18 to C17, C16 to C18, C17 to C19, C3 to C2, C4 to C3, C19 to C4, C2 to C5, C5 to C6, C6 to C7, C7 to C8, C8 to C9, J7 to J10, J10 to J3, J3 to J4, J4 to J5, J5 to J6, J6 to J7, J8 to J9, R8 to R10, R9 to R11, R10 to R12, R23 to R13, R24 to R14, R11 to R15, R12 to R16, R13 to R17, R14 to R3, R3 to R4, R4 to R5, R15 to R6, R5 to R7, R6 to R8, R7 to R9, SW3 to SW1
Connections:
- net DIR is gone; now on net DIR_1: J10.1 (Pin_1)
- net PWM is gone; now on net PWM_1: J10.2 (Pin_2)
- net En4_A_Tim4_CH1: now also U6.CN10_17 (PB6); no longer U6.CN10_4 (PC6)
- net En4_B_Tim4_CH2: now also U6.CN7_21 (PB7); no longer U6.CN10_19 (PC7)
- net FDCAN_1RX: now also U6.CN10_14 (PA11)
- net FDCAN_1TX: now also U6.CN10_12 (PA12)
- net FDCAN_2RX: now also U6.CN10_16 (PB12)
- net FDCAN_2TX: now also U6.CN10_30 (PB13)
- net GND: now also J11.3 (Pin_3), J8.2 (Pin_2), J8.3 (Pin_3)
- net PWM_servo: now also J8.1 (Pin_1)
- net board_num1: now also U6.CN7_38 (PC0/PB8)
- net board_num2: now also U6.CN7_36 (PC1/PB9)
- net DIR_1: now reaches U6.CN7_32 (PA4)
- net PWM_1: now reaches U6.CN7_34 (PB0)
- net DIR_2: now reaches U6.CN10_22 (PB2)
- net DIR_2: now also J11.1 (Pin_1)
- net PWM_2: now reaches U6.CN10_24 (PB1)
- net PWM_2: now also J11.2 (Pin_2)
- net En5_A_Tim5_CH1 renamed En5_A_Tim8_CH1
- net En5_A_Tim8_CH1: now also U6.CN10_4 (PC6); no longer U6.CN10_17 (PB6)
- net En5_B_Tim5_CH2 renamed En5_B_Tim8_CH2
- net En5_B_Tim8_CH2: now also U6.CN10_19 (PC7); no longer U6.CN7_21 (PB7)
- no-connect marks 5 -> 41
Other:
- moved on the sheet: C1, C10, C11, C12, C13, C14, C15, C16, C17, C2, C3, C4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
