File: SpringRobocon2026_mainboard.kicad_sch (KiCad schematic)
At the start: 68 parts, among them J1 Conn_01x05_Socket_Encoder1, J10 Conn_01x04_Pin, J11 Conn_01x03_Pin, J12 Conn_01x03_Pin, J2 Conn_01x05_Socket_Encoder3, J3 Conn_01x05_Socket_Encoder5, J4 FDCAN_1, J5 Conn_01x05_Socket_Encoder2, J6 Conn_01x05_Socket_Encoder4, J7 FDCAN_2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

Commit message: 修正完了
Parts:
- J9: value Conn_01x03_Pin -> Conn_01x02_Pin; footprint Connector_PinHeader_2.54mm:PinHeader_1x03_P2.54mm_Vertical -> Connector_PinHeader_2.54mm:PinHeader_1x02_P2.54mm_Vertical; symbol Connector:Conn_01x03_Pin -> Connector:Conn_01x02_Pin
- U3: value BP5293-50 -> BA50BC0FP; footprint MyLib:BP5293-xx_horizontal -> Package_TO_SOT_SMD:TO-252-2
Connections:
- net GND: no longer J9.3 (Pin_3)
Changed lines of the file:
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@@
 	)
 	(junction
-		(at 314.96 226.06)
-		(diameter 0)
-		(color 0 0 0 0)
-	)
-	(junction
 		(at 149.86 154.94)
 		(diameter 0)
@@
 	(wire
 		(pts
-			(xy 314.96 223.52) (xy 314.96 226.06)
-		)
-		(stroke
-			(width 0)
-			(type default)
-		)
-	)
-	(wire
-		(pts
 			(xy 318.77 175.26) (xy 318.77 177.8)
 		)
@@
 	(wire
 		(pts
-			(xy 314.96 220.98) (xy 309.88 220.98)
+			(xy 314.96 223.52) (xy 309.88 223.52)
 		)
 		(stroke
@@
 	(wire
 		(pts
-			(xy 309.88 223.52) (xy 314.96 223.52)
-		)
-		(stroke
-			(width 0)
-			(type default)
-		)
-	)
-	(wire
-		(pts
 			(xy 168.91 97.79) (xy 168.91 113.03)
 		)
@@
 	(global_label "PWM_servo"
 		(shape input)
-		(at 314.96 220.98 0)
+		(at 314.96 223.52 0)
 		(fields_autoplaced yes)
 		(effects
@@
 		)
 		(property "Intersheetrefs" "${INTERSHEET_REFS}"
-			(at 328.1051 220.98 0)
+			(at 328.1051 223.52 0)
 			(effects
 				(font
@@
 	)
 	(symbol
-		(lib_id "Connector:Conn_01x03_Pin")
+		(lib_id "Connector:Conn_01x02_Pin")
 		(at 304.8 223.52 0)
 		(unit 1)
@@
 		(fields_autoplaced yes)
 		(property "Reference" "J9"
-			(at 305.435 215.9 0)
+			(at 305.435 218.44 0)
 			(effects
 				(font
@@
 			)
 		)
-		(property "Value" "Conn_01x03_Pin"
-			(at 305.435 218.44 0)
+		(property "Value" "Conn_01x02_Pin"
+			(at 305.435 220.98 0)
 			(effects
 				(font
@@
 			)
 		)
-		(property "Footprint" "Connector_PinHeader_2.54mm:PinHeader_1x03_P2.54mm_Vertical"
+		(property "Footprint" "Connector_PinHeader_2.54mm:PinHeader_1x02_P2.54mm_Vertical"
 			(at 304.8 223.52 0)
 			(effects
@@
 			)
 		)
-		(property "Description" "Generic connector, single row, 01x03, script generated"
+		(property "Description" "Generic connector, single row, 01x02, script generated"
 			(at 304.8 223.52 0)
 			(effects
@@
 		(pin "2"
 		)
-		(pin "3"
-		)
 		(pin "1"
 		)
@@
 			)
 		)
-		(property "Value" "BP5293-50"
+		(property "Value" "BA50BC0FP"
 			(at 111.76 36.83 0)
 			(effects
@@
 			)
 		)
-		(property "Footprint" "MyLib:BP5293-xx_horizontal"
+		(property "Footprint" "Package_TO_SOT_SMD:TO-252-2"
 			(at 112.395 44.45 0)
 			(effects

Commit message: 一応のバックアップ
Parts:
- F1: value Polyfuse -> MF-NSMF035X; footprint Capacitor_THT:C_Disc_D8.0mm_W2.5mm_P5.00mm -> MyLib:PolyFuse_MF-NSMF-series
Changed lines of the file:
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@@
 		(on_board yes)
 		(dnp no)
-		(fields_autoplaced yes)
 		(property "Reference" "F1"
-			(at 71.12 35.56 90)
-			(effects
-				(font
-					(size 1.27 1.27)
-				)
-			)
-		)
-		(property "Value" "Polyfuse"
-			(at 71.12 38.1 90)
-			(effects
-				(font
-					(size 1.27 1.27)
-				)
-			)
-		)
-		(property "Footprint" "Capacitor_THT:C_Disc_D8.0mm_W2.5mm_P5.00mm"
+			(at 71.12 34.29 90)
+			(effects
+				(font
+					(size 1.27 1.27)
+				)
+			)
+		)
+		(property "Value" "MF-NSMF035X"
+			(at 71.12 36.83 90)
+			(effects
+				(font
+					(size 1.27 1.27)
+				)
+			)
+		)
+		(property "Footprint" "MyLib:PolyFuse_MF-NSMF-series"
 			(at 76.2 39.37 0)
 			(effects
@@
 		(dnp no)
 		(property "Reference" "D1"
-			(at 81.28 34.29 0)
+			(at 81.28 37.846 0)
 			(effects
 				(font
@@
 		)
 		(property "Value" "RB168MM100TR"
-			(at 81.28 36.83 0)
-			(effects
-				(font
+			(at 81.28 43.18 0)
+			(effects
+				(font
