File: SpringRobocon2026_mainboard.kicad_pcb (KiCad board)
At the start: 2 copper layers, 100 x 100 mm, 72 parts, among them J1 Conn_01x05_Socket_Encoder1, J10 Conn_01x04_Pin, J11 Conn_01x03_Pin, J12 Conn_01x03_Pin, J2 Conn_01x05_Socket_Encoder3, J3 Conn_01x05_Socket_Encoder5, J4 FDCAN_1, J5 Conn_01x05_Socket_Encoder2, J6 Conn_01x05_Socket_Encoder4, J7 FDCAN_2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

Commit message: 配置変更
Parts:
- moved R14 90.5 mm to (176.9, 49.7), turned to 180 degrees
- moved SW1 88.6 mm to (173.9, 49.7), turned to 0 degrees
- moved R16 86.9 mm to (176.8, 52.3), turned to 180 degrees
- moved J10 60.6 mm to (157.4, 113.8)
- moved D3 34.5 mm to (114.2, 99.2), turned to 180 degrees
- moved D9 29.9 mm to (149.0, 101.6), turned to 0 degrees
- moved C14 23.7 mm to (131.0, 107.5)
- moved C15 23.7 mm to (140.3, 107.6)
- moved C16 23.7 mm to (145.3, 106.7)
- moved U4 23.7 mm to (135.7, 111.0)
- moved D4 23.7 mm to (135.8, 103.4)
- moved D5 23.7 mm to (150.6, 108.0)
- moved R19 21.0 mm to (154.4, 103.7), turned to 90 degrees
- moved C7 20.8 mm to (119.2, 109.8)
- moved C8 20.8 mm to (119.2, 106.2)
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Routing:
- net +5V: track 97.4 -> 251.7 mm, vias 0 -> 6
- net +3V3: track 96.0 -> 182.9 mm, vias 6 -> 12
- net En2_B_Tim2_CH2: track 0.00 -> 47.5 mm
- net PWM_1: track 0.00 -> 9.98 mm
- net DIR_1: track 0.00 -> 9.96 mm
- net PWM_servo: track 0.00 -> 9.54 mm
- net Net-(D9-A): track 0.00 -> 3.32 mm
- net Net-(D1-A): track 5.37 -> 3.39 mm
- net +12V: track 31.2 -> 29.3 mm
- net En2_A_Tim2_CH1: track 0.00 -> 1.87 mm
- net Net-(D1-K): track 18.3 -> 16.8 mm
