File: SpringRobocon2026_mainboard.kicad_pcb (KiCad board)
At the start: 2 copper layers, 100 x 100 mm, 73 parts, among them J1 Conn_01x05_Socket_Encoder1, J10 Conn_01x04_Pin, J11 Conn_01x03_Pin, J12 Conn_01x03_Pin, J2 Conn_01x05_Socket_Encoder3, J3 Conn_01x05_Socket_Encoder5, J4 FDCAN_1, J5 Conn_01x05_Socket_Encoder2, J6 Conn_01x05_Socket_Encoder4, J7 FDCAN_2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

Commit message: 修正完了
Parts:
- J9: value Conn_01x03_Pin -> Conn_01x02_Pin; footprint Connector_PinHeader_2.54mm:PinHeader_1x03_P2.54mm_Vertical -> Connector_PinHeader_2.54mm:PinHeader_1x02_P2.54mm_Vertical
- U3: value BP5293-50 -> BA50BC0FP; footprint MyLib:BP5293-xx_horizontal -> Package_TO_SOT_SMD:TO-252-2; moved to B.Cu
- moved D3 12.9 mm to (127.0, 100.7)
- moved C9 11.6 mm to (127.0, 106.0), turned to 90 degrees
- moved U3 7.24 mm to (119.1, 111.0)
- moved J12 6.64 mm to (179.0, 79.5), turned to 180 degrees
- moved D2 6.61 mm to (119.5, 103.5), turned to 0 degrees
- moved J10 5.37 mm to (152.0, 113.5), turned to -90 degrees
- moved C7 5.24 mm to (114.5, 107.5), turned to -90 degrees
- moved C8 4.48 mm to (123.5, 107.5)
- moved C6 3.53 mm to (112.2, 110.0), turned to 180 degrees
- moved R19 1.21 mm to (153.5, 104.5)
Routing:
- net +5V: track 254.5 -> 292.1 mm, vias 6 -> 7
- net +3V3: track 183.3 -> 157.7 mm, vias 12 -> 6
- net DIR_2: track 8.56 -> 15.3 mm
- net SCL: track 61.5 -> 66.9 mm
- net PWM_2: track 8.65 -> 11.8 mm
- net En3_A_Tim3_CH1: track 48.9 -> 51.1 mm
- net En3_B_Tim3_CH2: track 40.4 -> 42.5 mm
- net GND: track 3.95 -> 1.92 mm, vias 919 -> 1011
- net En4_A_Tim4_CH1: track 63.8 -> 65.7 mm
- net SDA: track 61.5 -> 63.4 mm
- net En5_B_Tim8_CH2: track 41.5 -> 43.1 mm, vias 1 -> 0
- net FDCAN_2RX: track 31.1 -> 29.9 mm
- net En1_A_Tim1_CH1: track 43.1 -> 42.3 mm, vias 2 -> 1
- net En4_B_Tim4_CH2: track 65.1 -> 65.7 mm
- net En2_A_Tim2_CH1: track 65.9 -> 66.4 mm, vias 1 -> 3
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Other:
- board text added: "PWM GND"
- board text removed: "PWM GND GND"

Commit message: 一応のバックアップ
Parts:
- F1: value Polyfuse -> MF-NSMF035X; footprint Capacitor_THT:C_Disc_D8.0mm_W2.5mm_P5.00mm -> MyLib:PolyFuse_MF-NSMF-series; moved to B.Cu
- moved F1 2.99 mm to (105.5, 119.5)
Routing:
- net +5V: track 292.1 -> 295.2 mm
- net GND: vias 1011 -> 1016
Other:
- board text added: "L H"

Commit message: 再修正
Parts:
- moved D1 1.78 mm to (110.0, 115.5)
- moved D9 1.48 mm to (150.5, 101.8)
- moved R19 0.90 mm to (153.0, 105.2)
Routing:
- net +5V: track 295.2 -> 324.8 mm, vias 7 -> 13
- net +3V3: track 157.7 -> 171.2 mm
- net Net-(D1-A): track 3.39 -> 5.33 mm
- net Net-(D1-K): track 17.3 -> 16.7 mm
- net En2_B_Tim2_CH2: track 48.4 -> 48.6 mm, vias 0 -> 2
- net GND: vias 1016 -> 1007
